File: hardware/dmxduino/dmxduino.sch (KiCad schematic (older format))
At the start: 93 parts, among them J1 Conn_01x02, J10 Conn_01x02, J11 Conn_01x02, J2 Conn_01x02, J3 Conn_01x02, J4 Conn_01x01, J5 Conn_01x01, J6 Conn_01x01, J7 Conn_01x01, J8 Conn_01x02, J9 Conn_01x02, U1 LM324, U2 LM317_TO-220, U3 PC817, U4 LM317_TO-220, U5 LM324, U6 PC817, U7 PC817, U8 PC817, U9 LM324

Commit message: small improvements
Parts:
- removed J4, J5, J6, J7: Conn_01x01, symbol Connector_Generic:Conn_01x01
- removed J?: Conn_01x03, symbol Connector_Generic:Conn_01x03
- removed J?: Conn_01x09, symbol Connector_Generic:Conn_01x09
- removed R? (x2): R, symbol Device:R
- removed U?: PC817, Package_DIP:DIP-4_W7.62mm, symbol Isolator:PC817
- added J12: Conn_01x01_Male, Connector_PinHeader_2.54mm:PinHeader_1x01_P2.54mm_Vertical, symbol Connector:Conn_01x01_Male
- added J13: Conn_01x03_Female, Connector_PinHeader_2.54mm:PinHeader_1x03_P2.54mm_Vertical, symbol Connector:Conn_01x03_Female
- added J14: Conn_01x02, Connector_PinHeader_2.54mm:PinHeader_1x02_P2.54mm_Vertical, symbol Connector_Generic:Conn_01x02
- added J15, J16, J17, J18, J19, J20, J6, J7: Conn_01x02_Female, Connector_PinHeader_2.54mm:PinHeader_1x02_P2.54mm_Vertical, symbol Connector:Conn_01x02_Female
- added J24: Conn_01x02_Male, Connector_PinHeader_2.54mm:PinHeader_1x02_P2.54mm_Vertical, symbol Connector:Conn_01x02_Male
- added J25: Screw_Terminal_01x02, TerminalBlock:TerminalBlock_bornier-2_P5.08mm, symbol Connector:Screw_Terminal_01x02
- added J4: Conn_01x04_Male, Connector_PinHeader_2.54mm:PinHeader_1x04_P2.54mm_Vertical, symbol Connector:Conn_01x04_Male
- added J5: Conn_01x10_Female, Connector_PinHeader_2.54mm:PinHeader_1x10_P2.54mm_Vertical, symbol Connector:Conn_01x10_Female
- added K1: FINDER-36.11, Relay_THT:Relay_SPDT_Finder_36.11, symbol Relay:FINDER-36.11
- added Q1, Q2, Q3, Q4, Q5, Q6, Q7, Q8, Q9: 2N2219, Package_TO_SOT_THT:TO-92, symbol Transistor_BJT:2N2219
- added R47: 2k2, Resistor_THT:R_Axial_DIN0204_L3.6mm_D1.6mm_P7.62mm_Horizontal, symbol Device:R
- added R48: 47k, Resistor_THT:R_Axial_DIN0204_L3.6mm_D1.6mm_P7.62mm_Horizontal, symbol Device:R
- added R49, R50, R51, R52, R53, R54, R55, R56: 1k, Resistor_THT:R_Axial_DIN0204_L3.6mm_D1.6mm_P7.62mm_Horizontal, symbol Device:R
- added R57, R58, R59, R60, R61, R62, R63, R64: 47k, Resistor_THT:R_Axial_DIN0204_L3.6mm_D1.6mm_P2.54mm_Vertical, symbol Device:R
- C1, C10, C11, C12, C13, C3, C5, C6, C7, C9: footprint (none) -> Capacitor_THT:C_Disc_D7.5mm_W4.4mm_P5.00mm
- C14, C15, C16, C2, C4, C8: footprint (none) -> Capacitor_THT:CP_Radial_D10.0mm_P3.80mm
- J1, J10, J11, J2, J3, J8, J9: footprint (none) -> Connector_PinHeader_2.54mm:PinHeader_1x02_P2.54mm_Vertical
- R1, R10, R11, R12, R13, R14, R15, R16, R17, R18, R19, R2, R20, R21, R22, R23, R24, R25, R26, R27, R28, R29, R3, R30, R31, R32, R33, R34, R35, R36, R37, R38, R39, R4, R40, R41, R42, R43, R44, R45, R46, R5, R6, R7, R8, R9: footprint (none) -> Resistor_THT:R_Axial_DIN0204_L3.6mm_D1.6mm_P7.62mm_Horizontal
- RV1, RV2, RV3, RV4, RV5, RV6: footprint (none) -> Potentiometer_THT:Potentiometer_Bourns_3266Y_Vertical
- U1, U5, U9: footprint (none) -> Package_DIP:DIP-14_W7.62mm
Connections:
- net +12V: now also J13.1 (Pin_1), J24.1 (Pin_1), J25.1 (Pin_1)
- net +6V: now also U3.3, U5.10 (+), U5.12 (+), U5.5 (+), U9.10 (+), U9.12 (+), U9.5 (+); no longer R11.2, U5.10 (+), U5.12 (+), U5.5 (+), U9.10 (+), U9.12 (+), U9.5 (+)
- net +8.5V: now also R11.1; no longer U3.4
- net GND: now also J13.3 (Pin_3), J15.2 (Pin_2), J16.2 (Pin_2), J17.2 (Pin_2), J18.2 (Pin_2), J19.2 (Pin_2), J20.2 (Pin_2), J24.2 (Pin_2), J25.2 (Pin_2), J6.2 (Pin_2), J7.2 (Pin_2), Q1.1 (E), R48.2
- net PWM_0: now also J4.1 (Pin_1)
- net PWM_1: now also J4.2 (Pin_2)
- net PWM_2: now also J4.3 (Pin_3)
- net PWM_3: now also J4.4 (Pin_4)
- net at RV1.2, U1.3 (+): now also U1.5 (+); no longer U1.10 (+)
- net at C2.2, R1.1, R2.2: now also U1.13 (-); no longer U1.6 (-)
- net at C2.1, R2.1, R4.2: now also U1.14; no longer U1.7
- net at C3.1, R5.2, R8.2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: now also U1.7; no longer U1.8
- net at C3.2, RV5.2: now also U1.6 (-); no longer U1.9 (-)
- net at C4.2, R5.1, R6.2: now also U1.9 (-); no longer U1.13 (-)
- net at C4.1, R6.1, R7.2: now also U1.8; no longer U1.14
- net at C11.2, R29.2, R35.2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: now also U5.7; no longer U5.8
- net at C11.1, R32.1: now also U5.6 (-); no longer U5.9 (-)
- net at C14.1, R35.1, R38.2: now also U5.9 (-); no longer U5.13 (-)
- net at C14.2, R38.1, R42.2: now also U5.8; no longer U5.14
- net at C8.1, R17.1, R18.2: now also U5.13 (-); no longer U5.6 (-)
- net at C8.2, R18.1, R20.2: now also U5.14; no longer U5.7
- net at C15.1, R36.1, R39.2: now also U9.13 (-); no longer U9.6 (-)
- net at C15.2, R39.1, R44.2: now also U9.14; no longer U9.7
- net at C13.2, R31.2, R37.2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: now also U9.7; no longer U9.8
- net at C13.1, R34.1: now also U9.6 (-); no longer U9.9 (-)
- net at C16.1, R37.1, R40.2: now also U9.9 (-); no longer U9.13 (-)
- net at C16.2, R40.1, R46.2: now also U9.8; no longer U9.14
- new net: RV3.2, U1.10 (+), U1.12 (+)
- new net: R11.2, R12.2, U3.4
- new net: J5.10 (Pin_10), Q2.1 (E), R57.1
- new net: J5.3 (Pin_3), Q9.1 (E), R64.1
- new net: J5.4 (Pin_4), Q8.1 (E), R63.1
- new net: J5.5 (Pin_5), Q7.1 (E), R62.1
- new net: J5.6 (Pin_6), Q6.1 (E), R61.1
- new net: J5.7 (Pin_7), Q5.1 (E), R60.1
- new net: J5.8 (Pin_8), Q4.1 (E), R59.1
- new net: J5.9 (Pin_9), Q3.1 (E), R58.1
- new net: Q2.2 (B), R49.1, R57.2
- new net: J6.1 (Pin_1), Q2.3 (C)
- new net: J13.2 (Pin_2), K1.A1
- new net: Q1.2 (B), R47.1, R48.1
- new net: K1.A2, Q1.3 (C)
- new net: J12.1 (Pin_1), R47.2
- new net: J7.1 (Pin_1), Q3.3 (C)
- new net: Q3.2 (B), R50.1, R58.2
- new net: J15.1 (Pin_1), Q4.3 (C)
- new net: Q4.2 (B), R51.1, R59.2
- new net: J16.1 (Pin_1), Q5.3 (C)
- new net: Q5.2 (B), R52.1, R60.2
- new net: J17.1 (Pin_1), Q6.3 (C)
- new net: Q6.2 (B), R53.1, R61.2
- new net: J18.1 (Pin_1), Q7.3 (C)
- new net: Q7.2 (B), R54.1, R62.2
- new net: J19.1 (Pin_1), Q8.3 (C)
- new net: Q8.2 (B), R55.1, R63.2
- new net: J20.1 (Pin_1), Q9.3 (C)
- new net: Q9.2 (B), R56.1, R64.2
- new net: J14.1 (Pin_1), K1.11
- new net: J14.2 (Pin_2), K1.14
- new net +3V3: J5.1 (Pin_1), J5.2 (Pin_2), R49.2, R50.2, R51.2, R52.2, R53.2, R54.2, R55.2, R56.2
- no-connect marks 0 -> 1
Other:
- note added: "Adaptation niveau logique leds :\nInterface entre l'arduino (3.3V) et les leds (5V)"
- note added: "Commande logique"
- note added: "Commande manuelle"
- note added: "Sécurité alimentation laser"
- moved on the sheet: R11
